File: hardware/ioboard_2ports_rdm_isolated/ioboard_2ports_rdm_isolated.kicad_sch (KiCad schematic)
At the start: 33 parts, among them J1 Conn_02x06_Odd_Even, J12 Conn_01x03, J2 XLR3, J3 XLR3, J4 8P8C, J5 8P8C, J6 Conn_01x03, J8 XLR3, J9 XLR3, U1 M24C64-RMN6TP, U2 CRE1S0505DC, U4 ADM2483xRW, U6 ADM2483xRW

Commit message: Update all footprints and ignore all other DRC warning on ioboards
Parts:
- PS1: footprint Converter_DCDC:Converter_DCDC_muRata_CRE1xxxxxx3C_THT -> Converter_DCDC:Converter_DCDC_Murata_CRE1xxxxxx3C_THT
- U2: footprint Converter_DCDC:Converter_DCDC_muRata_CRE1xxxxxxDC_THT -> Converter_DCDC:Converter_DCDC_Murata_CRE1xxxxxxDC_THT
Changed lines of the file:
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@@
 			)
 		)
-		(property "Footprint" "Converter_DCDC:Converter_DCDC_muRata_CRE1xxxxxxDC_THT"
+		(property "Footprint" "Converter_DCDC:Converter_DCDC_Murata_CRE1xxxxxxDC_THT"
 			(at 186.69 36.83 0)
 			(effects
@@
 			)
 		)
-		(property "Footprint" "Converter_DCDC:Converter_DCDC_muRata_CRE1xxxxxx3C_THT"
+		(property "Footprint" "Converter_DCDC:Converter_DCDC_Murata_CRE1xxxxxx3C_THT"
 			(at 160.02 50.8 0)
 			(effects
